File: FanTimer.brd (EAGLE design)
At the start: 22 parts, among them IC2 NE555, T1 BT138-H

Commit message: del 817
Parts:
- added C4: (no value), rcl:C0805
- added D6, D7, D8, D9: (no value), diode:SOD80C
- added LINE1: (no value), DSS0:CON_PWR_2PIN4MM
- added OK1: PC817, optocoupler:DIL04
- added R10: (no value), rcl:0411/12
- added R7: 250, rcl:0207/10
- added R8, R9: (no value), rcl:R0805
- added T2: (no value), transistor:TO92-ECB
- added U$4: MOC3063MD, DSS0:DIL6
- added U$5: C, DSS0:C_22X10
- moved JP1 37.9 mm to (115.6, 8.89)
- moved R5 10.2 mm to (104.1, 73.7)
- moved U$3 10.2 mm to (104.1, 72.4)
- moved R6 1.27 mm to (82.5, 72.4)
Connections:
- removed net PE: C1.2, C2.-, C3.-, D3.A, D4.A, IC2.1, U$1.2, U$2.A
- new net -12V: C1.2, C2.-, C3.-, D3.A, D4.A, IC2.1, OK1.3, T2.E, U$2.A, U$4.2
- new net N$1: T2.C, U$1.2
- new net N$10: C4.2, D8.A, D9.A, OK1.2, R8.1
- new net N$15: OK1.4, R9.1, T2.B
- new net N$16: D6.A, D8.C, R10.2, U$5.2
- new net N$17: JP1.2, R10.1, U$5.1
- new net N$2: R6.2, U$4.4
- new net N$21: D7.A, D9.C, JP1.1
- new net N$22: C4.1, D6.C, D7.C, OK1.1, R8.2
- new net N$4: R7.2, U$4.1
- net +12V: now also R9.2
- net N$11: now also LINE1.2; no longer LINE.2
- net N$12: now also R7.1
- net N$18: now also U$4.6; no longer R6.2
Routing:
- net -12V: track 0.00 -> 90.4 mm, vias 0 -> 2
- net PE: track 83.7 -> 0.00 mm
- net N$4: track 0.00 -> 76.3 mm
- net N$10: track 0.00 -> 23.2 mm
- net N$11: track 27.7 -> 13.7 mm
- net N$13: track 15.3 -> 28.5 mm
- net +12V: track 94.6 -> 106.0 mm
- net N$12: track 7.40 -> 18.6 mm
- net N$16: track 0.00 -> 8.95 mm
- net N$18: track 0.00 -> 6.96 mm
- net N$14: track 18.0 -> 24.3 mm
- net N$15: track 0.00 -> 5.40 mm
- net N$1: track 0.00 -> 5.08 mm
- net LINE: track 38.4 -> 42.2 mm
- net N$2: track 0.00 -> 2.70 mm

Commit message: r1
Parts:
- removed C4: (no value), rcl:C0805
- removed D6, D7, D8, D9: (no value), diode:SOD80C
- removed JP1: (no value), pinhead:1X02
- removed LINE1: (no value), DSS0:CON_PWR_2PIN4MM
- removed R10: (no value), rcl:0411/12
- removed R6: (no value), rcl:R1206
- removed R8, R9: (no value), rcl:R0805
- removed U$5: C, DSS0:C_22X10
- added C5: (no value), rcl:C0805
- added D10, D11, D12: 1N4004, diode:DO41-10
- added N: (no value), DSS0:CON_PWR_2PIN4MM
- added R11, R12, R13: (no value), rcl:0207/10
- added RF1, RF2: (no value), rcl:R1206
- added T3: (no value), transistor:TO92-ECB
- moved OK1 77.3 mm to (149.9, 41.9), turned to 180 degrees
- moved D3 24.4 mm to (105.4, 82.5)
- moved U$4 15.5 mm to (86.4, 90.2)
- moved D2 15.3 mm to (116.8, 71.1), turned to 90 degrees
- moved U$2 9.92 mm to (108.0, 61.0)
- moved D4 9.92 mm to (97.8, 64.8)
- moved D5 9.16 mm to (108.0, 67.3)
- moved LINE 5.08 mm to (72.4, 71.1)
- moved R5 3.59 mm to (101.6, 76.2)
- moved U$3 2.84 mm to (101.6, 73.7)
- moved OUT 1.80 mm to (78.7, 59.7)
Connections:
- removed net N$10: C4.2, D8.A, D9.A, OK1.2, R8.1
- removed net N$11: D2.A, D3.C, LINE1.2, OUT.1
- removed net N$15: OK1.4, R9.1, T2.B
- removed net N$16: D6.A, D8.C, R10.2, U$5.2
- removed net N$17: JP1.2, R10.1, U$5.1
- removed net N$21: D7.A, D9.C, JP1.1
- removed net N$22: C4.1, D6.C, D7.C, OK1.1, R8.2
- new net N$20: D2.A, D3.C, R5.2, U$3.2
- new net N$23: R13.2, T3.B
- new net N$24: N.1, N.2, OUT.1, R5.1, U$3.1
- new net N$26: C5.1, R12.2, T2.B
- new net N$28: T3.C, U$1.2
- new net N$7: D11.C, D12.A, R12.1
- new net SWITCH: D10.C, D11.A, RF2.2
- net +12V: now also D12.C, R11.2; no longer R9.2
- net -12V: now also C5.2, D10.A, T3.E; no longer OK1.3
- net LINE: now also RF1.1; no longer R6.1
- net N$1: now also D4.C, D5.A, U$4.6; no longer T2.C, U$1.2
- net N$12: now also R7.2; no longer R7.1
- net N$14: now also R11.1, R13.1, T2.C; no longer D4.C, D5.A, R5.2, U$3.2
- net N$18: now also LINE.2, RF2.1; no longer R5.1, U$3.1, U$4.6
- net N$2: now also RF1.2; no longer R6.2
- net N$4: now also R7.1; no longer R7.2
Routing:
- net LINE: track 42.2 -> 0.00 mm
- net N$4: track 76.3 -> 42.4 mm
- net N$24: track 0.00 -> 27.0 mm
- net N$14: track 24.3 -> 0.00 mm
- net N$10: track 23.2 -> 0.00 mm
- net -12V: track 90.4 -> 70.2 mm, vias 2 -> 0
- net N$20: track 0.00 -> 17.6 mm
- net N$12: track 18.6 -> 3.59 mm
- net N$9: track 14.3 -> 0.00 mm
- net N$11: track 13.7 -> 0.00 mm
- net N$16: track 8.95 -> 0.00 mm
- net N$7: track 0.00 -> 7.62 mm
- net N$18: track 6.96 -> 0.00 mm
- net +12V: track 106.0 -> 99.1 mm
- net N$15: track 5.40 -> 0.00 mm
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
Commit message: .
Parts:
- removed OK1: PC817, optocoupler:DIL04
Connections:
- net LINE: no longer RF1.1
- net N$18: now also RF1.1
Changed lines of the file:
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@@
 <?xml version="1.0" encoding="utf-8"?>
 <!DOCTYPE eagle SYSTEM "eagle.dtd">
-<eagle version="6.4">
+<eagle version="6.3">
 <drawing>
 <settings>
@@
 <board>
 <plain>
-<dimension x1="60.96" y1="96.52" x2="128.27" y2="101.6" x3="94.615" y3="-13.97" textsize="3.5" layer="21" dtype="horizontal"/>
-<dimension x1="151.13" y1="58.42" x2="143.51" y2="63.5" x3="52.07" y3="60.96" textsize="3.5" layer="21" dtype="vertical"/>
+<dimension x1="60.96" y1="96.52" x2="128.27" y2="101.6" x3="94.615" y3="-13.97" layer="21" dtype="horizontal"/>
+<dimension x1="146.05" y1="5.08" x2="137.16" y2="95.25" x3="52.07" y3="50.165" layer="21" dtype="vertical"/>
 </plain>
 <attributes>
@@
 <element name="U$4" library="DSS0" package="DIL6" value="MOC3063MD" x="86.36" y="90.17" rot="R180"/>
 <element name="R7" library="rcl" package="0207/10" value="250" x="110.49" y="24.13"/>
-<element name="OK1" library="optocoupler" package="DIL04" value="PC817" x="149.86" y="41.91" rot="R180">
-<attribute name="OC_NEWARK" value="97K7059" x="149.86" y="41.91" size="1.778" layer="27" rot="R180" display="off"/>
-<attribute name="MPN" value="PC817X4J000F" x="149.86" y="41.91" size="1.778" layer="27" rot="R180" display="off"/>
-<attribute name="MF" value="" x="149.86" y="41.91" size="1.778" layer="27" rot="R180" display="off"/>
-<attribute name="OC_FARNELL" value="9707727" x="149.86" y="41.91" size="1.778" layer="27" rot="R180" display="off"/>
-</element>
 <element name="T2" library="transistor" package="TO92-ECB" value="" x="74.93" y="30.48" rot="R180"/>
 <element name="N" library="DSS0" package="CON_PWR_2PIN4MM" value="" x="74.93" y="82.55" rot="R270"/>
@@
 </signal>
 <signal name="LINE">
-<contactref element="RF1" pad="1"/>
 <contactref element="LINE" pad="1"/>
 <contactref element="R1" pad="2"/>
 <contactref element="T1" pad="T2"/>
-<wire x1="72.39" y1="73.12" x2="67.158" y2="87.63" width="0" layer="19" extent="16-16"/>
 <wire x1="69.85" y1="53.34" x2="72.39" y2="73.12" width="0" layer="19" extent="1-1"/>
 <wire x1="77.68636875" y1="49.9035" x2="69.85" y2="53.34" width="0" layer="19" extent="1-1"/>
@@
 <contactref element="LINE" pad="2"/>
 <contactref element="RF2" pad="1"/>
-<wire x1="72.39" y1="69.12" x2="78.588" y2="66.04" width="0" layer="19" extent="16-16"/>
+<contactref element="RF1" pad="1"/>
+<wire x1="72.39" y1="69.12" x2="67.158" y2="87.63" width="0" layer="19" extent="16-16"/>
+<wire x1="78.588" y1="66.04" x2="72.39" y2="69.12" width="0" layer="19" extent="16-16"/>
 </signal>
 <signal name="N$20">
